File: left/nrsk-left.kicad_sch (KiCad schematic)
At the start: 131 parts, among them J1 PJ-320D, J2 USB-C, J3 OLED 128x32, SW1 Esc, SW10 1, SW11 2, SW12 3, SW13 4, SW14 5, SW15 6, SW16 16, SW17 Tab, SW18 Q, SW19 W, SW2 F1, SW20 E, SW21 R, SW22 T, SW23 23, SW24 Ctrl, SW25 A, SW26 S, SW27 D, SW28 F, SW29 G, SW3 F2, SW30 30, SW31 Shift, SW32 Z, SW33 X, SW34 C, SW35 V, SW36 B, SW37 37, SW38 Ctrl, SW39 Opt, SW4 F3, SW40 Cmd, SW41 Space, SW42 Space, SW43 Space, SW44 44, SW5 F4, SW6 F5, SW7 F6, SW8 8, SW9 `, U1 RP2040, U2 USBLC6-2SC6, U3 AS5600-ASOM, U4 AP2112K-3.3, U5 W25Q128JVS, Y1 12MHz

Commit message: Schematic: thumbwheel encoder ENC1 on GP19 / GP20 instead of the AS5600 (spec step 2) - ENC1 (Device:RotaryEncoder, nrsk:Alps_EC05E1220401): A -> ENC_A -> GP19, B -> ENC_B -> GP20,   C -> GND; RP2040 internal pull-ups, so no resistors - U3 (AS5600), C9 (1 uF) and C10 (0.1 uF) removed, and with them the custom AS5600 symbol   (lib/nrsk.kicad_sym is empty now; the generator keeps the slot for later custom symbols) - layout.py: WHEEL_PIN_A / WHEEL_PIN_B; WHEEL_I2C_ADDR stays until the firmware step - Spec: pin pitch of the encoder lands corrected to 2.0 mm (the drawing's 3-1.5 is the land width) - Checked: ERC 0 violations on both halves; netlist has ENC1 A/B/C on /ENC_A (GPIO19),   /ENC_B (GPIO20) and GND, and no U3 / C9 / C10
Co-Authored-By: Claude Opus 5.5 <noreply@anthropic.com>
Parts:
- removed C10: 0.1uF, Capacitor_SMD:C_0805_2012Metric, symbol Device:C
- removed C9: 1uF, Capacitor_SMD:C_0805_2012Metric, symbol Device:C
- removed U3: AS5600-ASOM, Package_SO:SOIC-8_3.9x4.9mm_P1.27mm, symbol nrsk:AS5600
- added ENC1: EC05E1220401, nrsk:Alps_EC05E1220401, symbol Device:RotaryEncoder
Connections:
- net GND: now also ENC1.C
- net ENC_A: now reaches U1.30 (GPIO19)
- net ENC_A: now also ENC1.A
- net ENC_B: now reaches U1.31 (GPIO20)
- net ENC_B: now also ENC1.B
- no-connect marks 20 -> 16
Other:
- note added: "Thumbwheel encoder Alps EC05E1220401 (12 detents / 12 pulses, C = common)"
- note removed: "Thumbwheel sensor AS5600 (I2C 0x36, 3.3 V: VDD5V tied to VDD3V3)"
Changed lines of the file:
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@@
 	(label "COL6" (at 304.80 121.92 0) (effects (font (size 1.27 1.27)) (justify left bottom)))
 	(label "COL7" (at 304.80 124.46 0) (effects (font (size 1.27 1.27)) (justify left bottom)))
-	(no_connect (at 304.80 127.00))
-	(no_connect (at 304.80 129.54))
+	(label "ENC_A" (at 304.80 127.00 0) (effects (font (size 1.27 1.27)) (justify left bottom)))
+	(label "ENC_B" (at 304.80 129.54 0) (effects (font (size 1.27 1.27)) (justify left bottom)))
 	(no_connect (at 304.80 132.08))
 	(no_connect (at 304.80 134.62))
@@
 	(label "3V3" (at 378.46 209.55 90) (effects (font (size 1.27 1.27)) (justify left bottom)))
 	(label "SDA" (at 378.46 217.17 270) (effects (font (size 1.27 1.27)) (justify right bottom)))
-	(text "Thumbwheel sensor AS5600 (I2C 0x36, 3.3 V: VDD5V tied to VDD3V3)" (exclude_from_sim no) (at 330.20 236.22 0) (effects (font (size 2.0 2.0) (bold yes)) (justify left bottom)))
-	(symbol (lib_id "nrsk:AS5600") (at 342.90 254.00 0) (unit 1) (exclude_from_sim no) (in_bom yes) (on_board yes) (dnp no)
-	  (property "Reference" "U3" (at 345.44 251.46 0) (effects (font (size 1.27 1.27)) (justify left)))
-	  (property "Value" "AS5600-ASOM" (at 345.44 256.54 0) (effects (font (size 1.27 1.27)) (justify left)))
-	  (property "Footprint" "Package_SO:SOIC-8_3.9x4.9mm_P1.27mm" (at 342.90 254.00 0) (effects (font (size 1.27 1.27)) (hide yes)))
+	(text "Thumbwheel encoder Alps EC05E1220401 (12 detents / 12 pulses, C = common)" (exclude_from_sim no) (at 330.20 241.30 0) (effects (font (size 2.0 2.0) (bold yes)) (justify left bottom)))
+	(symbol (lib_id "Device:RotaryEncoder") (at 342.90 254.00 0) (unit 1) (exclude_from_sim no) (in_bom yes) (on_board yes) (dnp no)
+	  (property "Reference" "ENC1" (at 345.44 251.46 0) (effects (font (size 1.27 1.27)) (justify left)))
+	  (property "Value" "EC05E1220401" (at 345.44 256.54 0) (effects (font (size 1.27 1.27)) (justify left)))
+	  (property "Footprint" "nrsk:Alps_EC05E1220401" (at 342.90 254.00 0) (effects (font (size 1.27 1.27)) (hide yes)))
 	  (property "Datasheet" "" (at 342.90 254.00 0) (effects (font (size 1.27 1.27)) (hide yes)))
-	  (pin "1")
-	  (pin "2")
-	  (pin "3")
-	  (pin "4")
-	  (pin "5")
-	  (pin "6")
-	  (pin "7")
-	  (pin "8")
-	  (instances (project "nrsk-left" (path "/6c78887a-19a2-5291-a4e1-47e49dcf604a" (reference "U3") (unit 1))))
-	)
-	(label "3V3" (at 332.74 250.19 180) (effects (font (size 1.27 1.27)) (justify right bottom)))
-	(label "3V3" (at 332.74 252.73 180) (effects (font (size 1.27 1.27)) (justify right bottom)))
-	(no_connect (at 332.74 255.27))
-	(wire (pts (xy 332.74 257.81) (xy 327.66 257.81)) (stroke (width 0) (type default)))
-	(symbol (lib_id "power:GND") (at 327.66 257.81 270) (unit 1) (exclude_from_sim no) (in_bom no) (on_board no) (dnp no)
-	  (property "Reference" "#PWR043" (at 327.66 257.81 0) (effects (font (size 1.27 1.27)) (justify left) (hide yes)))
-	  (property "Value" "GND" (at 327.66 261.62 0) (effects (font (size 1.27 1.27)) (justify left)))
-	  (property "Footprint" "" (at 327.66 257.81 0) (effects (font (size 1.27 1.27)) (hide yes)))
-	  (property "Datasheet" "" (at 327.66 257.81 0) (effects (font (size 1.27 1.27)) (hide yes)))
+	  (pin "A")
+	  (pin "B")
+	  (pin "C")
+	  (instances (project "nrsk-left" (path "/6c78887a-19a2-5291-a4e1-47e49dcf604a" (reference "ENC1") (unit 1))))
+	)
+	(label "ENC_A" (at 335.28 251.46 180) (effects (font (size 1.27 1.27)) (justify right bottom)))
+	(label "ENC_B" (at 335.28 256.54 180) (effects (font (size 1.27 1.27)) (justify right bottom)))
+	(wire (pts (xy 335.28 254.00) (xy 330.20 254.00)) (stroke (width 0) (type default)))
+	(symbol (lib_id "power:GND") (at 330.20 254.00 270) (unit 1) (exclude_from_sim no) (in_bom no) (on_board no) (dnp no)
+	  (property "Reference" "#PWR043" (at 330.20 254.00 0) (effects (font (size 1.27 1.27)) (justify left) (hide yes)))
+	  (property "Value" "GND" (at 330.20 257.81 0) (effects (font (size 1.27 1.27)) (justify left)))
+	  (property "Footprint" "" (at 330.20 254.00 0) (effects (font (size 1.27 1.27)) (hide yes)))
+	  (property "Datasheet" "" (at 330.20 254.00 0) (effects (font (size 1.27 1.27)) (hide yes)))
 	  (pin "1")
 	  (instances (project "nrsk-left" (path "/6c78887a-19a2-5291-a4e1-47e49dcf604a" (reference "#PWR043") (unit 1))))
 	)
-	(no_connect (at 353.06 257.81))
-	(label "SDA" (at 353.06 255.27 0) (effects (font (size 1.27 1.27)) (justify left bottom)))
-	(label "SCL" (at 353.06 252.73 0) (effects (font (size 1.27 1.27)) (justify left bottom)))
-	(wire (pts (xy 353.06 250.19) (xy 358.14 250.19)) (stroke (width 0) (type default)))
-	(symbol (lib_id "power:GND") (at 358.14 250.19 90) (unit 1) (exclude_from_sim no) (in_bom no) (on_board no) (dnp no)
-	  (property "Reference" "#PWR044" (at 358.14 250.19 0) (effects (font (size 1.27 1.27)) (justify left) (hide yes)))
-	  (property "Value" "GND" (at 358.14 254.00 0) (effects (font (size 1.27 1.27)) (justify left)))
-	  (property "Footprint" "" (at 358.14 250.19 0) (effects (font (size 1.27 1.27)) (hide yes)))
-	  (property "Datasheet" "" (at 358.14 250.19 0) (effects (font (size 1.27 1.27)) (hide yes)))
-	  (pin "1")
-	  (instances (project "nrsk-left" (path "/6c78887a-19a2-5291-a4e1-47e49dcf604a" (reference "#PWR044") (unit 1))))
-	)
-	(symbol (lib_id "Device:C") (at 368.30 254.00 0) (unit 1) (exclude_from_sim no) (in_bom yes) (on_board yes) (dnp no)
-	  (property "Reference" "C9" (at 370.84 251.46 0) (effects (font (size 1.27 1.27)) (justify left)))
-	  (property "Value" "1uF" (at 370.84 256.54 0) (effects (font (size 1.27 1.27)) (justify left)))
-	  (property "Footprint" "Capacitor_SMD:C_0805_2012Metric" (at 368.30 254.00 0) (effects (font (size 1.27 1.27)) (hide yes)))
-	  (property "Datasheet" "" (at 368.30 254.00 0) (effects (font (size 1.27 1.27)) (hide yes)))
-	  (pin "1")
-	  (pin "2")
-	  (instances (project "nrsk-left" (path "/6c78887a-19a2-5291-a4e1-47e49dcf604a" (reference "C9") (unit 1))))
-	)
-	(label "3V3" (at 368.30 250.19 90) (effects (font (size 1.27 1.27)) (justify left bottom)))
-	(wire (pts (xy 368.30 257.81) (xy 368.30 262.89)) (stroke (width 0) (type default)))
-	(symbol (lib_id "power:GND") (at 368.30 262.89 0) (unit 1) (exclude_from_sim no) (in_bom no) (on_board no) (dnp no)
-	  (property "Reference" "#PWR045" (at 368.30 262.89 0) (effects (font (size 1.27 1.27)) (justify left) (hide yes)))
-	  (property "Value" "GND" (at 368.30 266.70 0) (effects (font (size 1.27 1.27)) (justify left)))
-	  (property "Footprint" "" (at 368.30 262.89 0) (effects (font (size 1.27 1.27)) (hide yes)))
-	  (property "Datasheet" "" (at 368.30 262.89 0) (effects (font (size 1.27 1.27)) (hide yes)))
-	  (pin "1")
-	  (instances (project "nrsk-left" (path "/6c78887a-19a2-5291-a4e1-47e49dcf604a" (reference "#PWR045") (unit 1))))
-	)
-	(symbol (lib_id "Device:C") (at 378.46 254.00 0) (unit 1) (exclude_from_sim no) (in_bom yes) (on_board yes) (dnp no)
-	  (property "Reference" "C10" (at 381.00 251.46 0) (effects (font (size 1.27 1.27)) (justify left)))
-	  (property "Value" "0.1uF" (at 381.00 256.54 0) (effects (font (size 1.27 1.27)) (justify left)))
-	  (property "Footprint" "Capacitor_SMD:C_0805_2012Metric" (at 378.46 254.00 0) (effects (font (size 1.27 1.27)) (hide yes)))
-	  (property "Datasheet" "" (at 378.46 254.00 0) (effects (font (size 1.27 1.27)) (hide yes)))
-	  (pin "1")
-	  (pin "2")
-	  (instances (project "nrsk-left" (path "/6c78887a-19a2-5291-a4e1-47e49dcf604a" (reference "C10") (unit 1))))
-	)
-	(label "3V3" (at 378.46 250.19 90) (effects (font (size 1.27 1.27)) (justify left bottom)))
-	(wire (pts (xy 378.46 257.81) (xy 378.46 262.89)) (stroke (width 0) (type default)))
-	(symbol (lib_id "power:GND") (at 378.46 262.89 0) (unit 1) (exclude_from_sim no) (in_bom no) (on_board no) (dnp no)
-	  (property "Reference" "#PWR046" (at 378.46 262.89 0) (effects (font (size 1.27 1.27)) (justify left) (hide yes)))
-	  (property "Value" "GND" (at 378.46 266.70 0) (effects (font (size 1.27 1.27)) (justify left)))
-	  (property "Footprint" "" (at 378.46 262.89 0) (effects (font (size 1.27 1.27)) (hide yes)))
-	  (property "Datasheet" "" (at 378.46 262.89 0) (effects (font (size 1.27 1.27)) (hide yes)))
-	  (pin "1")
-	  (instances (project "nrsk-left" (path "/6c78887a-19a2-5291-a4e1-47e49dcf604a" (reference "#PWR046") (unit 1))))
-	)
 	(sheet_instances (path "/" (page "1")))
